Commit message: depth_camera

File: description/robot.urdf.xacro (robot description, xacro)
@@ -2,4 +2,8 @@
 <robot xmlns:xacro="http://www.ros.org/wiki/xacro"  name="robot">
     <xacro:include filename="robot_core.xacro" />
-    <xacro:include filename="inertial_macros.xacro"/>
+    <xacro:include filename="ros2_control.xacro"/>
+    <!-- <xacro:include filename="gazebo_control.xacro"/> -->
+    <xacro:include filename="lidar.xacro"/>
+    <!-- <xacro:include filename="camera.xacro"/> -->
+    <xacro:include filename="depth_camera.xacro"/>
 </robot>

File: description/robot_core.xacro (robot description, xacro)
@@ -13,4 +13,7 @@
     <material name="blue">
         <color rgba="0.2 0.2 1 1"/>
+    </material>
+    <material name="red">
+        <color rgba="1 0 0 1"/>
     </material>
     <!-- base link-->
@@ -42,4 +45,7 @@
         </xacro:inertial_box>
     </link>
+    <gazebo reference="chassis">
+        <material>Gazebo/Orange</material>
+    </gazebo>
     <!-- left wheel link-->
     <joint name="left_wheel_joint" type="continuous">
@@ -66,4 +72,7 @@
         </xacro:inertial_cylinder>
     </link>
+    <gazebo reference="left_wheel">
+        <material>Gazebo/Black</material>
+    </gazebo>
     <!-- right wheel link-->
     <joint name="right_wheel_joint" type="continuous">
@@ -90,4 +99,7 @@
         </xacro:inertial_cylinder>
     </link>
+    <gazebo reference="right_wheel">
+        <material>Gazebo/Black</material>
+    </gazebo>
     <!-- caster wheel link -->
      <joint name="caster_wheel_joint" type="fixed">
@@ -113,3 +125,8 @@
         </xacro:inertial_sphere>
     </link>
+    <gazebo reference="caster_wheel">
+        <material>Gazebo/Blue</material>
+        <mu1 value="0.001"/>
+        <mu2 value="0.001"/>
+    </gazebo>
 </robot>
